File: Hardware/Schematics/SmartWatch.sch (KiCad schematic (older format))
At the start: 104 parts, among them J1 USB_C_Receptacle, J2 PIC32_ICSP, M1 Motor_DC, Q1 Photo_NPN, Q2 2N7000, SW1 SW_Push, SW2 SW_Push, U1 BQ25010, U2 PIC32MZ2048EFG064, U3 STMPE811, U4 nRF8001, U5 LSM303AGR, Y1 80MHz, Y2 32.768kHz, Y3 16MHz

Commit message: pin changes
Connections:
- net I2C_SCL: now also U2.6 (RPG8/SCL4/AN12); no longer U2.46 (INT0/RTCC/RPD0)
- net I2C_SDA: now also R15.1, U2.5 (RPG7/SDA4/AN13); no longer R15.2, U2.49 (SCK1/RPD1)
- net VCC: now also R15.2; no longer R15.1
- net BT_MISO renamed PGD
- net BT_MOSI renamed PGC
- net BT_SCK renamed SPI_SCK
Other:
- moved on the sheet: C16, C22, R15, R17
