File: Hardware/Schematics/_saved_SmartWatch.sch (KiCad schematic (older format))
At the start: 104 parts, among them J1 USB_C_Receptacle, J2 PIC32_ICSP, M1 Motor_DC, Q1 Photo_NPN, Q2 2N7000, SW1 SW_Push, SW2 SW_Push, U1 BQ25010, U2 PIC32MZ2048EFG064, U3 STMPE811, U4 nRF8001, U5 LSM303AGR, Y1 64MHz, Y2 32.768kHz, Y3 16MHz

Commit message: finish footprint selecting and started pcb
Parts:
- removed Y3: 16MHz, symbol Crystal
- added Y3: Crystal_GND24, 2450AT18A100E:CX2520DB16000F0FDFC1, symbol Crystal_GND24
- LCD1: footprint (none) -> 2450AT18A100E:NHD-1.8-128160EF-CTXI#-T
- Y1: footprint (none) -> Crystals:Crystal_SMD_HC49-SD_HandSoldering
- Y2: footprint (none) -> 2450AT18A100E:TFA322PG327KR
Connections:
- net GND: now also Y3.2, Y3.4
- net at C41.1, U4.~ (XC2): now also Y3.3
- net at C40.2, U4.~ (XC2): now also Y3.1
Changed lines of the file:
@@
 F 0 "Y2" H 5550 6050 50  0000 C CNN
 F 1 "32.768kHz" H 5700 5850 50  0000 C CNN
-F 2 "" H 5700 6000 50  0001 C CNN
+F 2 "2450AT18A100E:TFA322PG327KR" H 5700 6000 50  0001 C CNN
 F 3 "" H 5700 6000 50  0001 C CNN
 	1    5700 6000
@@
 F 0 "Y1" H 4900 6150 50  0000 C CNN
 F 1 "64MHz" H 4900 5850 50  0000 C CNN
-F 2 "" H 4900 6000 50  0001 C CNN
+F 2 "Crystals:Crystal_SMD_HC49-SD_HandSoldering" H 4900 6000 50  0001 C CNN
 F 3 "" H 4900 6000 50  0001 C CNN
 	1    4900 6000
@@
 NoConn ~ 11650 2550
 $Comp
-L Crystal Y3
-U 1 1 5A28E5E7
-P 11100 2200
-F 0 "Y3" H 10950 2250 50  0000 C CNN
-F 1 "16MHz" H 11100 2050 50  0000 C CNN
-F 2 "" H 11100 2200 50  0001 C CNN
-F 3 "" H 11100 2200 50  0001 C CNN
-	1    11100 2200
-	0    -1   -1   0
-$EndComp
-$Comp
 L C C41
 U 1 1 5A28EB88
@@
 F 0 "LCD1" H 2650 8050 59  0000 C CNN
 F 1 "NHD-1.8-128160EF-CTXI#-T" V 2900 6750 59  0000 C CNN
-F 2 "" H 2300 7800 59  0001 C CNN
+F 2 "2450AT18A100E:NHD-1.8-128160EF-CTXI#-T" H 2300 7800 59  0001 C CNN
 F 3 "" H 2300 7800 59  0001 C CNN
 	1    2650 6750
@@
 	10750 1950 10700 1950
 Wire Wire Line
-	10650 2200 10700 2200
+	10650 2200 10900 2200
 Connection ~ 10700 2200
 Wire Wire Line
@@
 	0    1    1    0
 $EndComp
+$Comp
+L Crystal_GND24 Y3
+U 1 1 5A5D5D30
+P 11100 2200
+F 0 "Y3" H 11225 2400 50  0000 L CNN
+F 1 "Crystal_GND24" V 10950 2350 50  0000 L CNN
+F 2 "2450AT18A100E:CX2520DB16000F0FDFC1" H 11100 2200 50  0001 C CNN
+F 3 "" H 11100 2200 50  0001 C CNN
+	1    11100 2200
+	0    1    1    0
+$EndComp
+$Comp
+L GND #PWR079
+U 1 1 5A5D666E
+P 11350 2200
+F 0 "#PWR079" H 11350 1950 50  0001 C CNN
+F 1 "GND" H 11350 2050 50  0000 C CNN
+F 2 "" H 11350 2200 50  0001 C CNN
+F 3 "" H 11350 2200 50  0001 C CNN
+	1    11350 2200
+	0    -1   -1   0
+$EndComp
+Wire Wire Line
+	11350 2200 11300 2200
 $EndSCHEMATC
