File: Hardware/Schematics/SmartWatch.kicad_pcb (KiCad board)
At the start: 2 copper layers, 104 parts, among them J1 USB_C_Receptacle, J2 PIC32_ICSP, M1 Motor_DC, Q1 Photo_NPN, Q2 2N7000, SW1 SW_Push, SW2 SW_Push, U1 BQ25010, U2 PIC32MZ2048EFG064, U3 STMPE811, U4 nRF8001, U5 LSM303AGR, Y1 64MHz, Y2 32.768kHz, Y3 Crystal_GND24

Commit message: Working on schematic
Parts:
- removed C27, C54, C56: 0.1uF, Capacitors_SMD:C_0805_HandSoldering
- removed C48: 100nF, Capacitors_SMD:C_0805_HandSoldering
- removed C49: 220nF, Capacitors_SMD:C_0805_HandSoldering
- removed C50: 22nF, Capacitors_SMD:C_0805_HandSoldering
- removed C51: 1.8pF, Capacitors_SMD:C_0805_HandSoldering
- removed C52: 10uF, Capacitors_SMD:C_0805_HandSoldering
- removed C53: 1.2pF, Capacitors_SMD:C_0805_HandSoldering
- removed C55: 1.5pF, Capacitors_SMD:C_0805_HandSoldering
- removed R23: 4k7, Resistors_SMD:R_0805_HandSoldering
- C1, C3: value 2pF -> 10pF; footprint Capacitors_SMD:C_0805_HandSoldering -> Capacitors_SMD:C_0603
- C10, C17: value 20pF -> 0.1uF; footprint Capacitors_SMD:C_0805_HandSoldering -> Capacitors_SMD:C_0603
- C11: value 0.1uF -> 10nF; footprint Capacitors_SMD:C_0805_HandSoldering -> Capacitors_SMD:C_0603
- C12, C24, C37, C9: footprint Capacitors_SMD:C_0805_HandSoldering -> Capacitors_SMD:C_0603
- C13, C20: value 0.1uF -> 1uF; footprint Capacitors_SMD:C_0805_HandSoldering -> Capacitors_SMD:C_0603
- C14: value 10uF -> 100nF; footprint Capacitors_SMD:C_0805_HandSoldering -> Capacitors_SMD:C_0603
- C15: value 10nF -> 33nF; footprint Capacitors_SMD:C_0805_HandSoldering -> Capacitors_SMD:C_0603
- C16: value 10uF -> 10nF; footprint Capacitors_SMD:C_0805_HandSoldering -> Capacitors_SMD:C_0603
- C18: value 0.1uF -> 22nF; footprint Capacitors_SMD:C_0805_HandSoldering -> Capacitors_SMD:C_0603
- C19: value 10nF -> 1uF; footprint Capacitors_SMD:C_0805_HandSoldering -> Capacitors_SMD:C_0603
- C2: value 0.1uF -> 1nF; footprint Capacitors_SMD:C_0805_HandSoldering -> Capacitors_SMD:C_0603
- C21, C25: value 10nF -> 0.1uF; footprint Capacitors_SMD:C_0805_HandSoldering -> Capacitors_SMD:C_0603
- C22, C26: value 0.1uF -> 10uF; footprint Capacitors_SMD:C_0805_HandSoldering -> Capacitors_SMD:C_0603
- C23: value 12.5pF -> 0.1uF; footprint Capacitors_SMD:C_0805_HandSoldering -> Capacitors_SMD:C_0603
- C28: value 12.5pF -> 20pF; footprint Capacitors_SMD:C_0805_HandSoldering -> Capacitors_SMD:C_0603
- C29: value 0.1uF -> 20pF; footprint Capacitors_SMD:C_0805_HandSoldering -> Capacitors_SMD:C_0603
- C30, C31: value 0.1uF -> 12.5pF; footprint Capacitors_SMD:C_0805_HandSoldering -> Capacitors_SMD:C_0603
- C32: value 10uF -> 220nF; footprint Capacitors_SMD:C_0805_HandSoldering -> Capacitors_SMD:C_0603
- C33: value 23pF -> 0.1uF; footprint Capacitors_SMD:C_0805_HandSoldering -> Capacitors_SMD:C_0603
- C34: value 0.15nF -> 10uF; footprint Capacitors_SMD:C_0805_HandSoldering -> Capacitors_SMD:C_0603
- C35: value 100nF -> 0.1uF; footprint Capacitors_SMD:C_0805_HandSoldering -> Capacitors_SMD:C_0603
- C36: value 1uF -> 23pF; footprint Capacitors_SMD:C_0805_HandSoldering -> Capacitors_SMD:C_0603
- C38: value 100nF -> 10uF; footprint Capacitors_SMD:C_0805_HandSoldering -> Capacitors_SMD:C_0603
- C39: value 33nF -> 100nF; footprint Capacitors_SMD:C_0805_HandSoldering -> Capacitors_SMD:C_0603
- C4: value 2pF -> 10nF; footprint Capacitors_SMD:C_0805_HandSoldering -> Capacitors_SMD:C_0603
- C40, C41: value 10pF -> 2pF; footprint Capacitors_SMD:C_0805_HandSoldering -> Capacitors_SMD:C_0603
- C42: value 0.1uF -> 0.15nF; footprint Capacitors_SMD:C_0805_HandSoldering -> Capacitors_SMD:C_0603
- C43: value 1uF -> 10uF; footprint Capacitors_SMD:C_0805_HandSoldering -> Capacitors_SMD:C_0603
- C44: value 1uF -> 0.1uF; footprint Capacitors_SMD:C_0805_HandSoldering -> Capacitors_SMD:C_0603
- C45: value 10uF -> 2pF; footprint Capacitors_SMD:C_0805_HandSoldering -> Capacitors_SMD:C_0603
- C46: value 0.1uF -> 2pF; footprint Capacitors_SMD:C_0805_HandSoldering -> Capacitors_SMD:C_0603
- C47: value 1nF -> 0.1uF; footprint Capacitors_SMD:C_0805_HandSoldering -> Capacitors_SMD:C_0603
- C5: value 10uF -> 0.1uF; footprint Capacitors_SMD:C_0805_HandSoldering -> Capacitors_SMD:C_0603
- C6: value 2pF -> 1.8pF; footprint Capacitors_SMD:C_0805_HandSoldering -> Capacitors_SMD:C_0603
- C7: value 10nF -> 1.2pF; footprint Capacitors_SMD:C_0805_HandSoldering -> Capacitors_SMD:C_0603
- C8: value 10nF -> 1.5pF; footprint Capacitors_SMD:C_0805_HandSoldering -> Capacitors_SMD:C_0603
- D1: value LED -> D; footprint LEDs:LED_0805_HandSoldering -> Diodes_SMD:D_0603
- D2: footprint LEDs:LED_0805_HandSoldering -> LEDs:LED_0603
- D3: value D -> LED; footprint Diodes_SMD:D_0805 -> LEDs:LED_0603
- J1: value USB_C_Receptacle -> PIC32_ICSP; footprint Connectors_USB:USB_C_Receptacle_Amphenol_12401548E4-2A_CircularHoles -> Pin_Headers:Pin_Header_Straight_2x03_Pitch1.00mm_SMD
- J2: value PIC32_ICSP -> USB_C_Receptacle; footprint Pin_Headers:Pin_Header_Straight_2x03_Pitch1.00mm_SMD -> Connectors_USB:USB_C_Receptacle_Amphenol_12401548E4-2A_CircularHoles
- L1: value 10uH -> 3.9nH; footprint Inductors_SMD:L_0805_HandSoldering -> Inductors_SMD:L_0603
- L2: footprint Inductors_SMD:L_0805_HandSoldering -> Inductors_SMD:L_0603
- L3: value 3.9nH -> 5.6nH; footprint Inductors_SMD:L_0805_HandSoldering -> Inductors_SMD:L_0603
- L4: value 5.6nH -> 10uH; footprint Inductors_SMD:L_0805_HandSoldering -> Inductors_SMD:L_0603
- Q1: value Photo_NPN -> 2N7000; footprint Diodes_SMD:D_3220 -> TO_SOT_Packages_THT:TO-92_Molded_Narrow
- Q2: value 2N7000 -> Photo_NPN; footprint TO_SOT_Packages_THT:TO-92_Molded_Narrow -> Diodes_SMD:D_3220
- R1: value 1M -> 10K; footprint Resistors_SMD:R_0805_HandSoldering -> Resistors_SMD:R_0603
- R10: value 1k -> 1M; footprint Resistors_SMD:R_0805_HandSoldering -> Resistors_SMD:R_0603
- R11: value 680k -> 1M; footprint Resistors_SMD:R_0805_HandSoldering -> Resistors_SMD:R_0603
- R12: value 121k -> 680k; footprint Resistors_SMD:R_0805_HandSoldering -> Resistors_SMD:R_0603
- R13, R14: value 100R -> 4k7; footprint Resistors_SMD:R_0805_HandSoldering -> Resistors_SMD:R_0603
- R15: value 4k7 -> 121k; footprint Resistors_SMD:R_0805_HandSoldering -> Resistors_SMD:R_0603
- R16: value 100k -> 1M; footprint Resistors_SMD:R_0805_HandSoldering -> Resistors_SMD:R_0603
- R17: value 4k7 -> 1k; footprint Resistors_SMD:R_0805_HandSoldering -> Resistors_SMD:R_0603
- R18, R19: footprint Resistors_SMD:R_0805_HandSoldering -> Resistors_SMD:R_0603
- R2: value 1M -> 470R; footprint Resistors_SMD:R_0805_HandSoldering -> Resistors_SMD:R_0603
- R20, R6: value 10k -> 100k; footprint Resistors_SMD:R_0805_HandSoldering -> Resistors_SMD:R_0603
- R21: value 22k -> 100R; footprint Resistors_SMD:R_0805_HandSoldering -> Resistors_SMD:R_0603
- R22: value 4k7 -> 100R; footprint Resistors_SMD:R_0805_HandSoldering -> Resistors_SMD:R_0603
- R3: value 100k -> 22k; footprint Resistors_SMD:R_0805_HandSoldering -> Resistors_SMD:R_0603
- R4: value 100k -> 4k7; footprint Resistors_SMD:R_0805_HandSoldering -> Resistors_SMD:R_0603
- R5: value 1M -> 4k7; footprint Resistors_SMD:R_0805_HandSoldering -> Resistors_SMD:R_0603
- R7: value 1M -> 100k; footprint Resistors_SMD:R_0805_HandSoldering -> Resistors_SMD:R_0603
- R8: value 10K -> 10k; footprint Resistors_SMD:R_0805_HandSoldering -> Resistors_SMD:R_0603
- R9: value 470R -> 1M; footprint Resistors_SMD:R_0805_HandSoldering -> Resistors_SMD:R_0603
- U1: value BQ25010 -> nRF8001; footprint Schematics:pvqfn-n20 -> Housings_DFN_QFN:QFN-32-1EP_5x5mm_Pitch0.5mm
- U3: value STMPE811 -> LSM303AGR; footprint Housings_DFN_QFN:QFN-20-1EP_4x4mm_Pitch0.5mm -> Housings_LGA:LGA-12_2x2mm_Pitch0.5mm
- U4: value nRF8001 -> STMPE811; footprint Housings_DFN_QFN:QFN-32-1EP_5x5mm_Pitch0.5mm -> Housings_DFN_QFN:QFN-20-1EP_4x4mm_Pitch0.5mm
- U5: value LSM303AGR -> BQ25010; footprint Housings_LGA:LGA-12_2x2mm_Pitch0.5mm -> Schematics:pvqfn-n20
- Y1: value 64MHz -> Crystal_GND24; footprint Crystals:Crystal_SMD_HC49-SD_HandSoldering -> 2450AT18A100E:CX2520DB16000F0FDFC1
- Y2: value 32.768kHz -> 64MHz; footprint 2450AT18A100E:TFA322PG327KR -> 2450AT18A100E:CX2520DB16000F0FDFC1
- Y3: value Crystal_GND24 -> 32.768kHz; footprint 2450AT18A100E:CX2520DB16000F0FDFC1 -> 2450AT18A100E:TFA322PG327KR
- moved Q1 175.1 mm to (219.1, 111.1), turned to 0 degrees
- moved Q2 172.7 mm to (192.4, 95.2)
- moved SW2 152.0 mm to (209.6, 115.6)
- moved C6 144.3 mm to (148.5, 105.0)
- moved ANT1 142.0 mm to (135.9, 41.9)
- moved C5 141.7 mm to (148.5, 105.0)
- moved U5 140.4 mm to (160.0, 41.9), turned to 180 degrees
- moved C4 139.3 mm to (148.5, 105.0)
- moved C12 138.9 mm to (148.5, 105.0)
- moved SW1 137.8 mm to (208.9, 121.9)
- moved C3 137.0 mm to (148.5, 105.0)
- moved C11 136.3 mm to (148.5, 105.0)
- moved C2 134.8 mm to (148.5, 105.0)
- moved C10 133.7 mm to (148.5, 105.0)
- moved C18 133.7 mm to (148.5, 105.0)
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Connections:
- C1 pad 1: LCD_YU -> GND
- C1 pad 2: GND -> Net-(C1-Pad2)
- C10 pad 1: Net-(C10-Pad1) -> VCC
- C11 pad 1: GND -> VCC
- C11 pad 2: VCC -> GND
- C13 pad 1: GND -> VCC
- C13 pad 2: VCC -> GND
- C14 pad 1: USB_VBUS -> Net-(C14-Pad1)
- C15 pad 1: VCC -> Net-(C15-Pad1)
- C16 pad 1: USB_VBUS -> GND
- C16 pad 2: GND -> VCC
- C17 pad 1: Net-(C17-Pad1) -> GND
- C17 pad 2: GND -> VCC
- C18 pad 1: USB_VBUS -> GND
- C18 pad 2: GND -> Net-(C18-Pad2)
- C19 pad 1: GND -> VCC
- C19 pad 2: VCC -> GND
- C2 pad 1: GND -> VCC
- C2 pad 2: VCC -> GND
- C20 pad 1: VCC -> GND
- C20 pad 2: GND -> VCC
- C21 pad 1: GND -> VCC
- C21 pad 2: VCC -> GND
- C22 pad 1: USB_VBUS -> GND
- C22 pad 2: GND -> VCC
- C23 pad 1: Net-(C23-Pad1) -> GND
- C23 pad 2: GND -> VCC
- C25 pad 1: VCC -> GND
- C25 pad 2: GND -> VCC
- C29 pad 1: AMB_LIGHT -> Net-(C29-Pad1)
- C3 pad 1: LCD_XL -> Net-(C3-Pad1)
- C30 pad 1: +BATT -> Net-(C30-Pad1)
- C31 pad 1: +BATT -> Net-(C31-Pad1)
- C32 pad 1: GND -> Net-(C32-Pad1)
- C32 pad 2: VCC -> GND
- C33 pad 2: Net-(C33-Pad2) -> GND
- C34 pad 1: Net-(C33-Pad2) -> GND
- C34 pad 2: GND -> VCC
- C35 pad 1: GND -> +BATT
- C35 pad 2: /VBAT_SENSE -> GND
- C36 pad 2: GND -> Net-(C36-Pad2)
- C38 pad 1: Net-(C38-Pad1) -> GND
- C38 pad 2: GND -> VCC
- C39 pad 1: Net-(C39-Pad1) -> VCC
- C39 pad 2: GND -> Net-(C39-Pad2)
- C4 pad 1: LCD_YD -> GND
- C4 pad 2: GND -> VCC
- C40 pad 1: GND -> LCD_YU
- C40 pad 2: Net-(C40-Pad2) -> GND
- C41 pad 1: Net-(C41-Pad1) -> LCD_YD
- C42 pad 1: VCC -> Net-(C36-Pad2)
- C43 pad 1: GND -> USB_VBUS
- C43 pad 2: VCC -> GND
- C44 pad 1: VCC -> USB_VBUS
- C45 pad 1: GND -> LCD_XL
- C45 pad 2: VCC -> GND
- C46 pad 1: VCC -> LCD_XR
- C47 pad 1: VCC -> AMB_LIGHT
- C6 pad 1: LCD_XR -> Net-(ANT1-Pad1)
- C6 pad 2: GND -> Net-(C6-Pad2)
- C7 pad 1: GND -> Net-(ANT1-Pad1)
- C7 pad 2: VCC -> GND
- C8 pad 1: VCC -> Net-(ANT1-Pad1)
- C9 pad 1: GND -> VCC
- C9 pad 2: VCC -> GND
- D1 pad 1: Net-(D1-Pad1) -> VCC
- D1 pad 2: LED1 -> Net-(C39-Pad2)
- D2 pad 2: LED2 -> LED1
- D3 pad 1: VCC -> Net-(D3-Pad1)
- D3 pad 2: Net-(C48-Pad2) -> LED2
- L1 pad 1: Net-(L1-Pad1) -> Net-(C6-Pad2)
- L1 pad 2: VCC -> Net-(L1-Pad2)
- L2 pad 1: Net-(L2-Pad1) -> Net-(L1-Pad2)
- L3 pad 1: Net-(C51-Pad2) -> Net-(C18-Pad2)
- L3 pad 2: Net-(L2-Pad1) -> Net-(L2-Pad2)
- L4 pad 1: Net-(C50-Pad2) -> Net-(L4-Pad1)
- L4 pad 2: Net-(L2-Pad2) -> VCC
- M1 pad 2: Net-(C48-Pad2) -> Net-(C39-Pad2)
- Q1 pad 1: VCC -> GND
- Q1 pad 2: AMB_LIGHT -> Net-(Q1-Pad2)
- Q2 pad 1: GND -> VCC
- Q2 pad 2: Net-(Q2-Pad2) -> AMB_LIGHT
- R1 pad 2: BAT_STAT1 -> Net-(J1-Pad1)
- R10 pad 1: Net-(R10-Pad1) -> VCC
- R10 pad 2: GND -> BAT_STAT1
- R11 pad 1: Net-(C33-Pad2) -> VCC
- R11 pad 2: VCC -> BAT_STAT2
- R12 pad 1: GND -> Net-(C36-Pad2)
- R12 pad 2: Net-(C33-Pad2) -> VCC
- R13 pad 2: Net-(D1-Pad1) -> Net-(Q1-Pad2)
- R14 pad 1: GND -> Net-(Q1-Pad2)
- R14 pad 2: Net-(D2-Pad1) -> MotorPWM
- R15 pad 1: VCC -> GND
- R15 pad 2: I2C_SCL -> Net-(C36-Pad2)
- R16 pad 1: GND -> BAT_CE
- R16 pad 2: /VBAT_SENSE -> GND
- R17 pad 1: VCC -> Net-(R17-Pad1)
- R17 pad 2: I2C_SDA -> GND
- R18 pad 1: /VBAT_SENSE -> GND
- R18 pad 2: +BATT -> BTN1
- R19 pad 1: VCC -> GND
- R19 pad 2: Net-(R19-Pad2) -> AMB_LIGHT
- R2 pad 1: VCC -> ~MCLR
- R2 pad 2: BAT_STAT2 -> Net-(J1-Pad1)
- R20 pad 1: VCC -> GND
- R20 pad 2: VCC -> BTN2
- R21 pad 2: Net-(R21-Pad2) -> Net-(D2-Pad1)
- R22 pad 1: Net-(Q2-Pad2) -> GND
- R22 pad 2: MotorPWM -> Net-(D3-Pad1)
- R3 pad 2: BTN1 -> Net-(R3-Pad2)
- R4 pad 1: GND -> VCC
- R4 pad 2: BTN2 -> I2C_SDA
- R5 pad 1: GND -> VCC
- R5 pad 2: Net-(R5-Pad2) -> I2C_SCL
- R6 pad 1: GND -> /VBAT_SENSE
- R6 pad 2: AMB_LIGHT -> +BATT
- R7 pad 1: BAT_CE -> GND
- R7 pad 2: GND -> /VBAT_SENSE
- R8 pad 2: Net-(J2-Pad1) -> Net-(R8-Pad2)
- R9 pad 1: ~MCLR -> GND
- R9 pad 2: Net-(J2-Pad1) -> Net-(R9-Pad2)
- U1 pad 1: (no net) -> VCC
- U1 pad 10: (no net) -> Net-(U1-Pad10)
- U1 pad 11: (no net) -> SPI_SCK
- U1 pad 12: Net-(R10-Pad1) -> BT_REQN
- U1 pad 13: +BATT -> PGC
- U1 pad 14: Net-(U1-Pad14) -> SPI_MOSI
- U1 pad 15: BAT_CE -> Net-(U1-Pad15)
- U1 pad 16: +BATT -> BT_RDYN
- U1 pad 17: +BATT -> GND
- U1 pad 19: Net-(L1-Pad1) -> BT_RESET
- U1 pad 2: Net-(C33-Pad2) -> Net-(C14-Pad1)
- U1 pad 20: GND -> Net-(C18-Pad2)
- U1 pad 21: (no net) -> Net-(L2-Pad2)
- U1 pad 3: GND -> Net-(C15-Pad1)
- U1 pad 4: +BATT -> Net-(U1-Pad4)
- U1 pad 5: Net-(R5-Pad2) -> Net-(U1-Pad5)
- U1 pad 6: USB_VBUS -> Net-(U1-Pad6)
- U1 pad 7: BAT_STAT1 -> Net-(U1-Pad7)
- U1 pad 8: BAT_STAT2 -> GND
- U1 pad 9: GND -> VCC
- U2 pad 31: Net-(C17-Pad1) -> Net-(C29-Pad1)
- U2 pad 32: Net-(C10-Pad1) -> Net-(C28-Pad1)
- U2 pad 47: Net-(C23-Pad1) -> Net-(C30-Pad1)
- U2 pad 48: Net-(C28-Pad1) -> Net-(C31-Pad1)
- U3 pad 1: LCD_YD -> I2C_SCL
- U3 pad 10: GND -> VCC
- U3 pad 11: Net-(U3-Pad11) -> INT2_XL
- U3 pad 12: Net-(U3-Pad12) -> INT1_XL
- U3 pad 2: Net-(R19-Pad2) -> VCC
- U3 pad 3: GND -> VCC
- U3 pad 4: I2C_SCL -> I2C_SDA
- U3 pad 5: I2C_SDA -> Net-(C32-Pad1)
- U3 pad 6: VCC -> GND
- U3 pad 7: VCC -> INT_MAG
- U3 pad 8: Net-(U3-Pad8) -> GND
- U3 pad 9: GND -> VCC
- U4 pad 1: VCC -> LCD_YD
- U4 pad 10: Net-(U4-Pad10) -> GND
- U4 pad 11: SPI_SCK -> Net-(U4-Pad11)
- U4 pad 12: BT_REQN -> Net-(U4-Pad12)
- U4 pad 13: PGC -> LCD_XL
- U4 pad 14: SPI_MOSI -> VCC
- U4 pad 15: Net-(U4-Pad15) -> LCD_YU
- U4 pad 16: BT_RDYN -> LCD_XR
- U4 pad 17: GND -> (no net)
- U4 pad 18: GND -> (no net)
- U4 pad 19: BT_RESET -> (no net)
- U4 pad 2: Net-(C38-Pad1) -> Net-(R8-Pad2)
- U4 pad 20: Net-(C50-Pad2) -> (no net)
- U4 pad 21: Net-(L2-Pad2) -> (no net)
- U4 pad 3: Net-(C39-Pad1) -> GND
- U4 pad 4: Net-(U4-Pad4) -> I2C_SCL
- U4 pad 5: Net-(U4-Pad5) -> I2C_SDA
- U4 pad 6: Net-(U4-Pad6) -> VCC
- U4 pad 7: Net-(U4-Pad7) -> VCC
- U4 pad 8: GND -> Net-(U4-Pad8)
- U4 pad 9: VCC -> GND
- U5 pad 1: I2C_SCL -> (no net)
- U5 pad 10: VCC -> (no net)
- U5 pad 11: INT2_XL -> (no net)
- U5 pad 12: INT1_XL -> Net-(R17-Pad1)
- U5 pad 2: VCC -> Net-(C36-Pad2)
- U5 pad 3: VCC -> GND
- U5 pad 4: I2C_SDA -> +BATT
- U5 pad 5: Net-(C49-Pad1) -> Net-(R9-Pad2)
- U5 pad 6: GND -> USB_VBUS
- U5 pad 7: INT_MAG -> BAT_STAT1
- U5 pad 8: GND -> BAT_STAT2
- U5 pad 9: VCC -> GND
- Y1 pad 1: Net-(C10-Pad1) -> Net-(C1-Pad2)
- Y1 pad 2: Net-(C17-Pad1) -> GND
- Y2 pad 1: Net-(C23-Pad1) -> Net-(C28-Pad1)
- Y2 pad 2: Net-(C28-Pad1) -> Net-(C29-Pad1)
- Y3 pad 1: Net-(C40-Pad2) -> Net-(C30-Pad1)
- Y3 pad 2: GND -> Net-(C31-Pad1)

Commit message: PCB
Parts:
- Y2: value 64MHz -> Crystal_GND24
- moved SW1 168.8 mm to (67.1, 30.5)
- moved SW2 161.3 mm to (67.6, 39.1)
- moved Q2 145.8 mm to (65.5, 23.4)
- moved Q1 145.8 mm to (91.4, 40.6)
- moved BT1 136.4 mm to (90.9, 23.9)
- moved M1 135.6 mm to (91.4, 32.0)
- moved J1 82.9 mm to (129.0, 25.4), turned to 0 degrees
- moved Y1 67.0 mm to (136.1, 39.1), turned to 180 degrees
- moved C1 64.7 mm to (100.6, 61.5)
- moved C10 64.7 mm to (100.6, 61.5)
- moved C11 64.7 mm to (100.6, 61.5)
- moved C12 64.7 mm to (100.6, 61.5)
- moved C13 64.7 mm to (100.6, 61.5)
- moved C14 64.7 mm to (100.6, 61.5)
- moved C15 64.7 mm to (100.6, 61.5)
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Connections:
- U1 pad 27: (no net) -> Net-(C1-Pad2)
- U1 pad 28: (no net) -> Net-(C3-Pad1)
- U1 pad 29: (no net) -> VCC
- U1 pad 30: (no net) -> GND
- U1 pad 31: (no net) -> GND
- U1 pad 32: (no net) -> Net-(U1-Pad32)
- U2 pad 33: (no net) -> USB_VBUS
- Y2 pad 1: Net-(C28-Pad1) -> Net-(C29-Pad1)
- Y2 pad 2: Net-(C29-Pad1) -> GND
- Y2 pad 3: (no net) -> Net-(C28-Pad1)
- Y2 pad 4: (no net) -> GND

Commit message: cant remember
Parts:
- BT1: footprint Pin_Headers:Pin_Header_Straight_2x01_Pitch2.54mm_SMD -> Pin_Headers:Pin_Header_Straight_2x01_Pitch2.54mm
- J1: footprint Pin_Headers:Pin_Header_Straight_2x03_Pitch1.00mm_SMD -> Pin_Headers:Pin_Header_Straight_2x03_Pitch2.54mm
- moved C18 168.3 mm to (265.8, 29.5), turned to 270 degrees
- moved C8 167.1 mm to (263.8, 25.7)
- moved C7 166.8 mm to (263.8, 27.0)
- moved L3 166.1 mm to (263.8, 30.3), turned to 180 degrees
- moved C6 164.7 mm to (261.6, 27.0), turned to 270 degrees
- moved L2 164.5 mm to (262.4, 31.8)
- moved L1 164.1 mm to (261.6, 29.8), turned to 270 degrees
- moved C2 161.8 mm to (259.5, 30.9), turned to 180 degrees
- moved C15 161.7 mm to (261.0, 40.8), turned to 270 degrees
- moved R3 161.6 mm to (259.5, 32.2)
- moved C14 160.5 mm to (259.7, 40.8), turned to 270 degrees
- moved C13 159.2 mm to (258.4, 41.2), turned to 270 degrees
- moved C3 158.2 mm to (257.0, 38.0), turned to 180 degrees
- moved C1 157.1 mm to (255.6, 35.6), turned to 90 degrees
- moved R10 137.8 mm to (231.0, 105.7), turned to 180 degrees
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Connections:
- U1 pad 33: (no net) -> GND
- U2 pad 56: Net-(U2-Pad56) -> T_INT
- U4 pad 2: Net-(R8-Pad2) -> T_INT
- U5 pad 21: (no net) -> GND
Routing:
- net GND: track 0.00 -> 35.5 mm
- net VCC: track 0.00 -> 15.9 mm
- net Net-(ANT1-Pad1): track 0.00 -> 7.14 mm
- net Net-(C1-Pad2): track 0.00 -> 6.87 mm
- net Net-(C36-Pad2): track 0.00 -> 5.80 mm
- net Net-(C18-Pad2): track 0.00 -> 5.45 mm
- net +BATT: track 0.00 -> 3.93 mm
- net BAT_STAT2: track 0.00 -> 3.92 mm
- net BAT_STAT1: track 0.00 -> 3.11 mm
- net Net-(C14-Pad1): track 0.00 -> 2.91 mm
- net Net-(U1-Pad32): track 0.00 -> 2.71 mm
- net Net-(L4-Pad1): track 0.00 -> 2.68 mm
- net USB_VBUS: track 0.00 -> 2.35 mm
- net Net-(R3-Pad2): track 0.00 -> 2.30 mm
- net Net-(L2-Pad2): track 0.00 -> 2.24 mm
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